File: flex/flex.kicad_pcb (KiCad board)
At the start: 2 copper layers, 104.1 x 90.6 mm, 105 parts, among them J1 Conn_01x04_Female, J2 Conn_01x05_Female, J3 Conn_01x03_Female, J4 Conn_01x06_Female, J5 Conn_01x03_Female, SW10 NA_SW_Push, SW11 NA_SW_Push, SW12 NA_SW_Push, SW15 NA_SW_Push, SW16 NA_SW_Push, SW17 NA_SW_Push, SW20 NA_SW_Push, SW21 NA_SW_Push, SW22 NA_SW_Push, SW24 NA_SW_Push, SW25 NA_SW_Push, SW26 NA_SW_Push, SW6 NA_SW_Push, SW7 NA_SW_Push, SW8 NA_SW_Push

Commit message: routing
Routing:
- net row2: track 0.00 -> 379.8 mm
- net row4: track 0.00 -> 318.9 mm
- net row3: track 0.00 -> 300.5 mm, vias 0 -> 1
- net col2: track 0.00 -> 228.3 mm, vias 0 -> 2
- net col6: track 0.00 -> 159.9 mm, vias 0 -> 2
- net col3: track 0.00 -> 145.6 mm, vias 0 -> 2
- net col5: track 0.00 -> 132.2 mm, vias 0 -> 3
- net Net-(D70-A): track 0.00 -> 70.2 mm, vias 0 -> 1
- net Net-(D31-A): track 0.00 -> 65.1 mm, vias 0 -> 3
- net Net-(D1-A): track 0.00 -> 64.5 mm, vias 0 -> 1
- net Net-(D17-A): track 0.00 -> 64.2 mm, vias 0 -> 1
- net Net-(D15-A): track 0.00 -> 44.6 mm, vias 0 -> 1
- net Net-(D19-A): track 0.00 -> 38.0 mm, vias 0 -> 1
- net Net-(D30-A): track 0.00 -> 35.3 mm, vias 0 -> 1
- net Net-(D14-A): track 0.00 -> 31.9 mm, vias 0 -> 1
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
Commit message: routing
Parts:
- moved D9 0.50 mm to (59.4, 87.8)
- moved D15 0.41 mm to (59.3, 111.8)
Connections:
- D42 pad 1: Net-(D42-DOUT) -> Net-(D41-DOUT)
- D48 pad 3: Net-(D42-DOUT) -> Net-(D41-DOUT)
Routing:
- net Net-(D25-DOUT): track 0.00 -> 134.2 mm, vias 0 -> 2
- net Gnd: track 0.00 -> 131.8 mm, vias 0 -> 16
- net Net-(D21-DIN): track 0.00 -> 118.5 mm, vias 0 -> 3
- net Vcc: track 0.00 -> 118.0 mm, vias 0 -> 17
- net Net-(D5-DIN): track 0.00 -> 103.1 mm, vias 0 -> 4
- net col4: track 30.8 -> 119.4 mm, vias 1 -> 3
- net Net-(D20-A): track 0.00 -> 73.9 mm, vias 0 -> 5
- net col2: track 228.3 -> 297.4 mm, vias 2 -> 6
- net row5: track 0.00 -> 59.2 mm
- net Net-(D27-A): track 0.00 -> 58.2 mm, vias 0 -> 4
- net col5: track 132.2 -> 185.7 mm, vias 3 -> 5
- net Net-(D37-DOUT): track 0.00 -> 53.4 mm, vias 0 -> 2
- net Net-(D23-DOUT): track 0.00 -> 43.2 mm, vias 0 -> 2
- net Net-(D21-DOUT): track 0.00 -> 41.1 mm, vias 0 -> 4
- net Net-(D33-DIN): track 0.00 -> 40.0 mm, vias 0 -> 3
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
Commit message: routing
Routing:
- net Gnd: track 131.8 -> 750.0 mm, vias 16 -> 29
- net Vcc: track 118.0 -> 700.7 mm, vias 17 -> 36
- net Net-(D41-DOUT): track 11.3 -> 128.8 mm, vias 2 -> 3
- net Net-(D51-DOUT): track 15.4 -> 104.1 mm, vias 2 -> 3
- net Net-(D49-DOUT): track 12.9 -> 71.1 mm, vias 2 -> 3
- net row4: track 326.3 -> 378.6 mm, vias 0 -> 3
- net Net-(D47-DOUT): track 11.9 -> 55.4 mm, vias 2 -> 3
- net Net-(D39-DOUT): track 11.5 -> 51.4 mm, vias 2 -> 4
- net row2: track 390.3 -> 429.6 mm
- net Net-(D55-DOUT): track 14.8 -> 48.0 mm
- net row3: track 307.3 -> 338.8 mm
- net Net-(D57-DOUT): track 12.3 -> 43.2 mm
- net Net-(D25-DOUT): track 134.2 -> 152.1 mm
- net Dout: track 4.37 -> 21.5 mm
- net col2: track 297.4 -> 314.5 mm
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
Commit message: routing
Routing:
- net Gnd: track 750.0 -> 769.7 mm
- net Vcc: track 700.7 -> 720.2 mm
- net row4: track 378.6 -> 396.7 mm
- net row2: track 429.6 -> 446.3 mm
- net row3: track 338.8 -> 354.6 mm
- net Net-(D21-DIN): track 118.5 -> 132.8 mm
- net col2: track 314.5 -> 327.9 mm
- net col6: track 190.5 -> 199.7 mm
- net Net-(D5-DIN): track 103.1 -> 94.7 mm, vias 4 -> 5
- net col5: track 199.5 -> 206.2 mm
- net Net-(D20-A): track 75.6 -> 81.8 mm
- net Net-(D41-DOUT): track 128.8 -> 133.6 mm
- net col3: track 179.1 -> 183.0 mm
- net Net-(D30-A): track 36.8 -> 40.5 mm
- net Net-(D51-DOUT): track 104.1 -> 107.6 mm
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